File: KiCad_Files/axolotl.kicad_sch (KiCad schematic)
At the start: 6 parts

Commit message: modifed pcb and updtaed tracks, footprints and fill-zones
Parts:
- BT1: value (none) -> Battery_Cell; footprint (none) -> Binary_Kitchen:BatteryHolder_Keystone_1060_1x2032_HandSoldering
- D1, D2, D3, D4: value (none) -> LED; footprint (none) -> Binary_Kitchen:5mm_SMD-Pad
- SW1: value (none) -> SW_DIP_x01; footprint (none) -> Binary_Kitchen:Push_Button
